Commit message: camera fixed

File: robots/descriptions/go2_description/urdf/go2_description.urdf (robot description, URDF)
Before this commit: robot go2_description, 39 links, 38 joints
Joints:
- joint camera_joint: origin xyz=0.285 0 0.08 rpy=0 0 0 -> xyz=0.285 0 0.08 rpy=0 1.22 0

File: robots/descriptions/go2_description/xacro/robot.xacro (robot description, xacro)
@@ -152,6 +152,6 @@
         <parent link="camera_bottom_screw_frame"/>
         <child link="camera_link"/>
-        <!-- Tilt camera slightly downward so the ground enters the FOV in simulation -->
-        <origin xyz="0 0.0175 0.0125" rpy="0 -0.35 0"/>
+        <!-- Camera pointing straight forward -->
+        <origin xyz="0 0.0175 0.0125" rpy="0 0 0"/>
     </joint>
     <joint name="camera_depth_joint" type="fixed">
