Commit message: map and other updates

File: robots/descriptions/go2_description/xacro/robot.xacro (robot description, xacro)
@@ -152,5 +152,6 @@
         <parent link="camera_bottom_screw_frame"/>
         <child link="camera_link"/>
-        <origin xyz="0 0.0175 0.0125" rpy="0 0 0"/>
+        <!-- Tilt camera slightly downward so the ground enters the FOV in simulation -->
+        <origin xyz="0 0.0175 0.0125" rpy="0 -0.35 0"/>
     </joint>
     <joint name="camera_depth_joint" type="fixed">
@@ -303,6 +304,7 @@
             <infrared1OpticalframeName>camera_left_ir_optical_frame</infrared1OpticalframeName>
             <infrared2OpticalframeName>camera_right_ir_optical_frame</infrared2OpticalframeName>
-            <rangeMinDepth>0.3</rangeMinDepth>
-            <rangeMaxDepth>3.0</rangeMaxDepth>
+            <!-- Extend valid depth range to reduce zero-depth frames in empty scenes -->
+            <rangeMinDepth>0.1</rangeMinDepth>
+            <rangeMaxDepth>20.0</rangeMaxDepth>
             <pointCloud>true</pointCloud>
             <pointCloudTopicName>depth/color/points</pointCloudTopicName>

Commit message: changes and updates to odometry plus maps

File: robots/descriptions/go2_description/xacro/robot.xacro (robot description, xacro)
@@ -7,4 +7,6 @@
     <!-- <xacro:include filename="$(find go2_description)/xacro/stairs.xacro"/> -->
     <xacro:include filename="$(find go2_description)/xacro/gazebo.xacro"/>
+    <!-- Livox LiDAR -->
+    <xacro:include filename="$(find ros2_livox_simulation)/urdf/mid70.xacro"/>
     <!-- <xacro:include filename="$(find go2_gazebo)/launch/stairs.urdf.xacro"/> -->
     <!-- <xacro:stairs stairs="15" xpos="0" ypos="0" zpos="0" /> -->
@@ -312,3 +314,7 @@
         </plugin>
     </gazebo>
+    <!-- Livox mid70 LiDAR mounted on top of the robot (lightest option - 10K samples) -->
+    <xacro:mid70 name="livox" parent="trunk" topic="/livox/lidar">
+        <origin xyz="0.0 0 0.15" rpy="0 0 0"/>
+    </xacro:mid70>
 </robot>
